File: electronics/vanarebane_version/view_base/view_base.kicad_pcb (KiCad board)
At the start: 2 copper layers, 81.2 x 81.2 mm, 122 parts, among them J1 BLDC, J2 USB_C_Receptacle_USB2.0, J3 LCD, J4 A, J5 B, Q1 MMBT4403, Q2 UMH3N, U1 MT6701-CT, U10 LM386, U11 VCNL4010-GS08, U2 T-Micro32_Plus, U3 CH340C, U4 HX711, U5 TMC6300, U6 AP2114HA-3.3, U7 SN74LV1T34DBV, U8 VEML7700, U9 TS1117BCW33_RPG

Commit message: Fix TMC_VL wired to input-only IO35: move to IO4
TMC6300 VL gate input was routed to ESP32 IO35 (GPIO34-39 have no output
driver), so the V-phase low-side FET could never be driven. Move TMC_VL
to IO4 (previously LCD_RST; firmware already uses TFT_RST=-1), tie LCD
reset to 3V3, reroute PCB (new B.Cu track, dead VL stub removed, zones
refilled) and update firmware pin map (PIN_VL=4, PIN_BUTTON_NEXT=0).

Co-Authored-By: Claude Fable 5.1 <noreply@anthropic.com>
Connections:
- J3 pad 3: /LCD_RST -> +3.3V
- U2 pad 26: /LCD_RST -> /TMC_VL
- U2 pad 7: /TMC_VL -> (no net)
Routing:
- net /TMC_VL: track 75.7 -> 115.6 mm, vias 2 -> 3
- net +3.3V: track 373.3 -> 380.7 mm
- net /LCD_RST: track 4.00 -> 0.00 mm, vias 1 -> 0
- net GND: vias 49 -> 48
