File: electronics/vanarebane_version/view_base/view_base.kicad_sch (KiCad schematic)
At the start: 122 parts, among them J1 BLDC, J2 USB_C_Receptacle_USB2.0, J3 LCD, J4 A, J5 B, Q1 MMBT4403, Q2 UMH3N, U1 MT6701-CT, U10 LM386, U11 VCNL4010-GS08, U2 T-Micro32_Plus, U3 CH340C, U4 HX711, U5 TMC6300, U6 AP2114HA-3.3, U7 SN74LV1T34DBV, U8 VEML7700, U9 TS1117BCW33_RPG

Commit message: Fix TMC_VL wired to input-only IO35: move to IO4
TMC6300 VL gate input was routed to ESP32 IO35 (GPIO34-39 have no output
driver), so the V-phase low-side FET could never be driven. Move TMC_VL
to IO4 (previously LCD_RST; firmware already uses TFT_RST=-1), tie LCD
reset to 3V3, reroute PCB (new B.Cu track, dead VL stub removed, zones
refilled) and update firmware pin map (PIN_VL=4, PIN_BUTTON_NEXT=0).

Co-Authored-By: Claude Fable 5.1 <noreply@anthropic.com>
Connections:
- net +3.3V: now also J3.3 (Pin_3)
- net TMC_VL: now also U2.26 (IO4); no longer U2.7 (IO35)
- removed net LCD_RST: J3.3 (Pin_3), U2.26 (IO4)
- no-connect marks 34 -> 35
Other:
- note added: "IO35 is input-only:"
- note added: "LCD reset via SW (TFT_RST=-1)"
- note added: "LCD_RST (J3.3) tied to 3V3;"
- note added: "TMC_VL moved to IO4"
Changed lines of the file:
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@@
   (junction (at 30.48 99.06) (diameter 0) (color 0 0 0 0)
   )
+  (text "IO35 is input-only:" (at 303.53 55.88 0)
+    (effects (font (size 1.016 1.016)) (justify left bottom))
+  )
+  (text "TMC_VL moved to IO4" (at 303.53 58.42 0)
+    (effects (font (size 1.016 1.016)) (justify left bottom))
+  )
+  (text "LCD_RST (J3.3) tied to 3V3;" (at 226.06 97.79 0)
+    (effects (font (size 1.016 1.016)) (justify left bottom))
+  )
+  (text "LCD reset via SW (TFT_RST=-1)" (at 226.06 100.33 0)
+    (effects (font (size 1.016 1.016)) (justify left bottom))
+  )
+  (no_connect (at 340.36 48.26))
   (no_connect (at 132.08 43.18))
   (no_connect (at 389.89 109.22))
@@
     (stroke (width 0) (type default) (color 0 0 0 0))
   )
-  (wire (pts (xy 340.36 48.26) (xy 325.12 48.26))
-    (stroke (width 0) (type default) (color 0 0 0 0))
-  )
   (wire (pts (xy 351.79 215.9) (xy 347.98 215.9))
     (stroke (width 0) (type default) (color 0 0 0 0))
@@
     (stroke (width 0) (type default) (color 0 0 0 0))
   )
-  (wire (pts (xy 242.57 80.01) (xy 226.06 80.01))
+  (wire (pts (xy 242.57 80.01) (xy 236.22 80.01))
     (stroke (width 0) (type default) (color 0 0 0 0))
   )
@@
     (effects (font (size 1.27 1.27)) (justify right bottom))
   )
-  (label "LCD_RST" (at 226.06 80.01 0)
-    (effects (font (size 1.27 1.27)) (justify left bottom))
-  )
   (label "TMC_VL" (at 180.34 135.89 0)
     (effects (font (size 1.27 1.27)) (justify left bottom))
@@
     (effects (font (size 1.27 1.27)) (justify left bottom))
   )
-  (label "LCD_RST" (at 394.97 63.5 180)
+  (label "TMC_VL" (at 394.97 63.5 180)
     (effects (font (size 1.27 1.27)) (justify right bottom))
   )
@@
     (effects (font (size 1.27 1.27)) (justify right bottom))
   )
-  (label "TMC_VL" (at 325.12 48.26 0)
-    (effects (font (size 1.27 1.27)) (justify left bottom))
-  )
   (label "LCD_SCK" (at 394.97 58.42 180)
     (effects (font (size 1.27 1.27)) (justify right bottom))
@@
     (pin "2")
   )
+  (symbol (lib_id "power:+3.3V") (at 236.22 80.01 0) (unit 1)
+    (in_bom yes) (on_board yes)
+    (property "Reference" "#PWR0162" (id 0) (at 236.22 83.82 0)
+      (effects (font (size 1.27 1.27)) hide)
+    )
+    (property "Value" "+3.3V" (id 1) (at 236.601 75.6158 0))
+    (property "Footprint" "" (id 2) (at 236.22 80.01 0)
+      (effects (font (size 1.27 1.27)) hide)
+    )
+    (property "Datasheet" "" (id 3) (at 236.22 80.01 0)
+      (effects (font (size 1.27 1.27)) hide)
+    )
+    (pin "1")
+  )
   (symbol (lib_id "power:+3.3V") (at 36.83 25.4 0) (unit 1)
     (in_bom yes) (on_board yes)
@@
       (reference "U1") (unit 1) (value "MT6701-CT") (footprint "Package_SO:SOIC-8_3.9x4.9mm_P1.27mm")
     )
+    (path "/e840e43b-2b4a-47fe-a67d-9e02f1542589"
+      (reference "#PWR0162") (unit 1) (value "+3.3V") (footprint "")
+    )
     (path "/00000000-0000-0000-0000-00006200e46e"
